Commit message: .

File: omni_wheel_description/xacro/omni_150mm.xacro (robot description, xacro)
@@ -27,4 +27,5 @@
     <xacro:property name="damping" value="1"/>
     <xacro:property name="friction" value="1"/>
+    <xacro:property name="collision_mesh_scaler" value="0.05"/>
     <!-- create the wheel link first -->
     <link name="${name}">
@@ -40,5 +41,5 @@
         <collision>
             <geometry>
-                <cylinder radius="${radius}" length="${width}"/>
+                <cylinder radius="${radius}" length="${width*collision_mesh_scaler}"/>
             </geometry>
         </collision>
